Commit message: Sensors fusion done!

File: src/urdf-model-v2_description/urdf/urdf-model-v2.xacro (robot description, xacro)
@@ -84,4 +84,24 @@
   </collision>
 </link>
+<link name="imu_1">
+  <inertial>
+    <origin rpy="0 0 0" xyz="-2.871335190220503e-07 -2.203098814490545e-16 0.001500000000000043"/>
+    <mass value="0.0033390000000000078"/>
+    <inertia ixx="0.0" ixy="0.0" ixz="-0.0" iyy="0.0" iyz="-0.0" izz="1e-06"/>
+  </inertial>
+  <visual>
+    <origin rpy="0 0 0" xyz="-4.7e-05 0.0105 -0.1195"/>
+    <geometry>
+      <mesh filename="package://urdf-model-v2_description/meshes/imu_1.stl" scale="0.001 0.001 0.001"/>
+    </geometry>
+    <material name="silver"/>
+  </visual>
+  <collision>
+    <origin rpy="0 0 0" xyz="-4.7e-05 0.0105 -0.1195"/>
+    <geometry>
+      <mesh filename="package://urdf-model-v2_description/meshes/imu_1.stl" scale="0.001 0.001 0.001"/>
+    </geometry>
+  </collision>
+</link>
 <joint name="Rev10" type="continuous">
   <origin rpy="0 0 0" xyz="0.0 0.1915 0.0465"/>
@@ -101,3 +121,8 @@
   <child link="lidar_1"/>
 </joint>
+<joint name="Rigid13" type="fixed">
+  <origin rpy="0 0 0" xyz="4.7e-05 -0.0105 0.1195"/>
+  <parent link="base_link"/>
+  <child link="imu_1"/>
+</joint>
 </robot>
